Commit message: feat: added random parcours to env

File: obstacles/my-simple-object.urdf (robot description, URDF)
Before this commit: robot obstacle, 1 links, 0 joints
Links:
- link base_link: geometry collision mesh filename=my-simple-object.stl scale=1 1 1; visual mesh filename=my-simple-object.stl scale=1 1 1
